Commit message: Updated readme, Sim Approach and others

File: gelsight_simulation/models/setup.xacro (robot description, xacro)
@@ -4,4 +4,5 @@
     <xacro:include filename="$(find gelsight_simulation)/models/solid.xacro"/>
     <xacro:arg name="solid_name" default="torus"/>
+    <xacro:arg name="rotation_rad" default="0"/>
     <xacro:solid name="$(arg solid_name)"/>
     <joint name="hook_gelsight_printer" type="fixed">
@@ -11,5 +12,5 @@
     </joint>
     <joint name="hook_solid" type="fixed">
-        <!--        <origin xyz="-0.045 0 0" rpy="0 0 ${pi/2}"/>-->
+        <origin xyz="0 0 0" rpy="0 0 $(arg rotation_rad)"/>
         <parent link="fdm_printer_bed"/>
         <child link="solid_link"/>
